Commit message: added macro

File: src/wheel_chair/description/urdf/wheel_chair_description_gazebo.urdf.xacro (robot description, xacro)
@@ -1,4 +1,5 @@
 <?xml version="1.0"?>
 <robot name="wheel_chair" xmlns:xacro="http://ros.org/wiki/xacro">
+  <xacro:macro name="wheel_chair" params="prefix">
 <!-- Define robot constants -->
   <xacro:property name="base_width" value="0.50"/>

Commit message: more xacro

File: src/wheel_chair/description/urdf/wheel_chair_description_gazebo.urdf.xacro (robot description, xacro)
@@ -364,2 +364,3 @@
 </gazebo>
 </robot>
+</xacro:macro>

Commit message: Revert "more xacro"
This reverts commit 520def4d3201567c7498e3ba7da50fe53212e51a.

File: src/wheel_chair/description/urdf/wheel_chair_description_gazebo.urdf.xacro (robot description, xacro)
@@ -364,3 +364,2 @@
 </gazebo>
 </robot>
-</xacro:macro>

Commit message: Revert "added macro"
This reverts commit 4961c90e855fccd0626f6ccf9d649402178f1509.

File: src/wheel_chair/description/urdf/wheel_chair_description_gazebo.urdf.xacro (robot description, xacro)
@@ -1,5 +1,4 @@
 <?xml version="1.0"?>
 <robot name="wheel_chair" xmlns:xacro="http://ros.org/wiki/xacro">
-  <xacro:macro name="wheel_chair" params="prefix">
 <!-- Define robot constants -->
   <xacro:property name="base_width" value="0.50"/>
