Commit message: edited xacro description

File: src/wheel_chair/description/urdf/wheel_chair_description.urdf.xacro (robot description, xacro)
@@ -3,13 +3,13 @@
   <xacro:macro name="wheel_chair" params="prefix">
 <!-- Define robot constants -->
-  <xacro:property name="base_width" value="0.51"/>
+  <xacro:property name="base_width" value="0.50"/>
   <xacro:property name="base_length" value="0.62"/>
-  <xacro:property name="base_height" value="0.18"/>
-  <xacro:property name="wheel_radius" value="0.10"/>
-  <xacro:property name="wheel_width" value="0.04"/>
+  <xacro:property name="base_height" value="0.05"/>
+  <xacro:property name="wheel_radius" value="0.095"/>
+  <xacro:property name="wheel_width" value="0.07"/>
   <xacro:property name="wheel_ygap" value="0.025"/>
   <xacro:property name="wheel_zoff" value="0.05"/>
-  <xacro:property name="wheel_xoff" value="0.12"/>
-  <xacro:property name="caster_xoff" value="0.14"/>
+  <xacro:property name="wheel_xoff" value="0.21"/>
+  <xacro:property name="caster_xoff" value="0.21"/>
   <!-- Define intertial property macros  -->
   <xacro:macro name="box_inertia" params="m w h d">
@@ -103,4 +103,22 @@
     <origin xyz="${caster_xoff} 0.0 ${-(base_height/2)}" rpy="0 0 0"/>
   </joint>
+<link name="imu_link">
+  <visual>
+    <geometry>
+      <box size="0.1 0.1 0.1"/>
+    </geometry>
+  </visual>
+  <collision>
+    <geometry>
+      <box size="0.1 0.1 0.1"/>
+    </geometry>
+  </collision>
+  <xacro:box_inertia m="0.1" w="0.1" d="0.1" h="0.1"/>
+</link>
+<joint name="imu_joint" type="fixed">
+  <parent link="base_link"/>
+  <child link="imu_link"/>
+  <origin xyz="0 0 0.01"/>
+</joint>
   </xacro:macro>
 </robot>

Commit message: remove imu link and spell check

File: src/wheel_chair/description/urdf/wheel_chair_description.urdf.xacro (robot description, xacro)
@@ -103,4 +103,5 @@
     <origin xyz="${caster_xoff} 0.0 ${-(base_height/2)}" rpy="0 0 0"/>
   </joint>
+<!--
 <link name="imu_link">
   <visual>
@@ -120,5 +121,5 @@
   <child link="imu_link"/>
   <origin xyz="0 0 0.01"/>
-</joint>
+</joint> -->
   </xacro:macro>
 </robot>
